File: HandyPad-main/PCB/Macropad from hackpad.kicad_pcb (KiCad board)
At the start: 2 copper layers, 53.9 x 77 mm, 17 parts, among them SW1 RotaryEncoder_Switch, SW2 SW_Push, SW3 SW_Push, SW4 SW_Push, SW5 SW_Push, SW6 SW_Push, SW8 SW_Push, SW9 SW_Push, U1 MOUDLE-SEEEDUINO-XIAO, U2 ER_OLEDM0.91_1x-I2C

Commit message: feat: update project details for Samrath "Sami" Singh
Co-authored-by: Sami.s <191058343+Sami9889@users.noreply.github.com>
Other:
- board text added: "SamiPad"
- board text added: "Samrath "Sami" Singh"
- board text added: "github.com/Sami9889"
Changed lines of the file:
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@@
 	)
 	(paper "A4")
+	(title_block
+		(title "SamiPad Macropad")
+		(company "Samrath \"Sami\" Singh")
+		(comment 1 "github.com/Sami9889")
+		(comment 2 "hackpad.hackclub.com")
+	)
 	(layers
 		(0 "F.Cu" signal)
@@
 			(drillshape 0)
 			(scaleselection 1)
-			(outputdirectory "C:/Users/nilay/Downloads/")
+			(outputdirectory "")
 		)
 	)
@@
 		)
 		(embedded_fonts no)
-		(model "C:/Users/nilay/Downloads/MX .STEP"
+		(model "${KIPRJMOD}/models/MX .STEP"
 			(offset
 				(xyz -9.9 -12.5 6)
@@
 		)
 		(embedded_fonts no)
-		(model "C:/Users/nilay/Downloads/MX .STEP"
+		(model "${KIPRJMOD}/models/MX .STEP"
 			(offset
 				(xyz -9.9 -12.5 6)
@@
 		)
 		(embedded_fonts no)
-		(model "C:/Users/nilay/Downloads/MX .STEP"
+		(model "${KIPRJMOD}/models/MX .STEP"
 			(offset
 				(xyz -9.9 -12.5 6)
@@
 		)
 		(embedded_fonts no)
-		(model "C:/Users/nilay/Downloads/EC11_Rotary_Encoder_Switched.step"
+		(model "${KIPRJMOD}/models/EC11_Rotary_Encoder_Switched.step"
 			(offset
 				(xyz 7.5 -2.5 0)
@@
 		)
 		(embedded_fonts no)
-		(model "C:/Users/nilay/Downloads/OLED_0.91_128x32.stp"
+		(model "${KIPRJMOD}/models/OLED_0.91_128x32.stp"
 			(offset
 				(xyz 4 -17.5 0)
@@
 		)
 		(embedded_fonts no)
-		(model "C:/Users/nilay/Downloads/MX .STEP"
+		(model "${KIPRJMOD}/models/MX .STEP"
 			(offset
 				(xyz -9.9 -12.5 6)
@@
 		)
 		(embedded_fonts no)
-		(model "C:/Users/nilay/Downloads/MX .STEP"
+		(model "${KIPRJMOD}/models/MX .STEP"
 			(offset
 				(xyz -9.9 -12.5 6)
@@
 		)
 		(embedded_fonts no)
-		(model "C:/Users/nilay/Downloads/MX .STEP"
+		(model "${KIPRJMOD}/models/MX .STEP"
 			(offset
 				(xyz -9.9 -12.5 6)
@@
 		)
 		(embedded_fonts no)
-		(model "C:/Users/nilay/Downloads/MX .STEP"
+		(model "${KIPRJMOD}/models/MX .STEP"
 			(offset
 				(xyz -9.9 -12.5 6)
@@
 		)
 		(embedded_fonts no)
-		(model "C:/Users/nilay/Downloads/Seeed Studio XIAO RP2040 v26.step"
+		(model "${KIPRJMOD}/models/Seeed Studio XIAO RP2040 v26.step"
 			(offset
 				(xyz 0 0 0)
@@
 		(net "Net-(D10-K)")
 	)
+	(gr_text "Samrath \"Sami\" Singh"
+		(at 111.75 143.2 0)
+		(layer "F.SilkS")
+		(effects
+			(font
+				(size 1.2 1.2)
+				(thickness 0.2)
+			)
+			(justify center bottom)
+		)
+	)
+	(gr_text "github.com/Sami9889"
+		(at 111.75 72.5 0)
+		(layer "B.SilkS")
+		(effects
+			(font
+				(size 1 1)
+				(thickness 0.15)
+			)
+			(justify center top mirror)
+		)
+	)
+	(gr_text "SamiPad"
+		(at 111.75 75.2 0)
+		(layer "B.SilkS")
+		(effects
+			(font
+				(size 1.4 1.4)
+				(thickness 0.25)
+			)
+			(justify center top mirror)
+		)
+	)
 	(embedded_fonts no)
