File: HandyPad-main/PCB/Macropad from hackpad.kicad_sch (KiCad schematic)
At the start: 17 parts, among them SW1 RotaryEncoder_Switch, SW2 SW_Push, SW3 SW_Push, SW4 SW_Push, SW5 SW_Push, SW6 SW_Push, SW8 SW_Push, SW9 SW_Push, U1 MOUDLE-SEEEDUINO-XIAO, U2 ER_OLEDM0.91_1x-I2C

Commit message: feat: update project details for Samrath "Sami" Singh
Co-authored-by: Sami.s <191058343+Sami9889@users.noreply.github.com>
Other:
- company: (none) -> Samrath "Sami" Singh
- title: (none) -> SamiPad Macropad
Changed lines of the file:
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@@
 	(generator_version "10.0")
 	(paper "A4")
+	(title_block
+		(title "SamiPad Macropad")
+		(company "Samrath \"Sami\" Singh")
+		(comment 1 "github.com/Sami9889")
+		(comment 2 "hackpad.hackclub.com")
+	)
 	(junction
 		(at 128.27 118.11)
